File: RouterSupplySwitcherSource/RouterSupplySwitcherSource.kicad_sch (KiCad schematic)
At the start: 0 parts

Commit message: added scheme
Parts:
- added C1, C2, C3, C4: C, symbol Device:C
- added D1, D2: D, symbol Device:D
- added D3: D_Schottky_Dual_CommonAnode_AKK_Split, CustomFootprintsLib:SS34, symbol Device:D_Schottky_Dual_CommonAnode_AKK_Split
- added J1, J2: Barrel_Jack_Switch, symbol Connector:Barrel_Jack_Switch
- added J3: USB_A, symbol Connector:USB_A
- added L1: L, symbol Device:L
- added P1: USB_C_Plug, symbol Connector:USB_C_Plug
- added R1: R, symbol Device:R
- added RV1: R_Potentiometer, symbol Device:R_Potentiometer
- added VR1: XL6009, CustomFootprintsLib:XL6009, symbol customLib:XL6009
Connections:
- new net: C3.1, C4.1, D3.2 (K), J2.1, J3.1 (VBUS), RV1.2, RV1.3
- new net: C1.2, C2.1, C3.2, C4.2, J1.2, J2.2, J3.4 (GND), P1.A1 (GND), P1.A12 (GND), P1.B1 (GND), P1.B12 (GND), R1.2, VR1.1 (GND)
- new net: D3.1 (A), L1.2, VR1.3 (SW), VR1.6 (SW)
- new net: C1.1, C2.2, D1.1 (K), D2.1 (K), L1.1, VR1.2 (EN), VR1.4 (VIN)
- new net: R1.1, RV1.1, VR1.5 (FB)
- new net: D1.2 (A), J1.1
- new net: D2.2 (A), P1.A4 (VBUS), P1.A9 (VBUS), P1.B4 (VBUS), P1.B9 (VBUS)
- no-connect marks 0 -> 20
