File: RouterSupplySwitcherSource/RouterSupplySwitcherSource.kicad_sch (KiCad schematic)
At the start: 15 parts, among them J1 Barrel_Jack_Switch, J2 Barrel_Jack_Switch, J3 USB_A, P1 USB_C_Plug

Commit message: added pcb
Parts:
- C1, C4: footprint Capacitor_THT:C_Radial_D4.0mm_H5.0mm_P1.50mm -> Capacitor_THT:CP_Radial_D4.0mm_P2.00mm
Changed lines of the file:
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@@
 			)
 		)
-		(property "Footprint" "Capacitor_THT:C_Radial_D4.0mm_H5.0mm_P1.50mm"
+		(property "Footprint" "Capacitor_THT:CP_Radial_D4.0mm_P2.00mm"
 			(at 171.1452 116.84 0)
 			(effects
@@
 			)
 		)
-		(property "Footprint" "Capacitor_THT:C_Radial_D4.0mm_H5.0mm_P1.50mm"
+		(property "Footprint" "Capacitor_THT:CP_Radial_D4.0mm_P2.00mm"
 			(at 100.0252 118.11 0)
 			(effects

Commit message: added values
Parts:
- C1: value C -> 220uF
- C2, C3: value C -> 0.1uF
- C4: value C -> 100uF
- D3: value D_Schottky_Dual_CommonAnode_AKK_Split -> SS34
- L1: value L -> 47uH
- R1: value R -> 330R
- RV1: value R_Potentiometer -> 10kR
Changed lines of the file:
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@@
 			)
 		)
-		(property "Value" "C"
+		(property "Value" "100uF"
 			(at 173.99 114.2999 0)
 			(effects
@@
 			)
 		)
-		(property "Value" "D_Schottky_Dual_CommonAnode_AKK_Split"
+		(property "Value" "SS34"
 			(at 153.924 91.44 0)
 			(effects
@@
 			)
 		)
-		(property "Value" "C"
+		(property "Value" "0.1uF"
 			(at 111.76 120.6499 0)
 			(effects
@@
 			)
 		)
-		(property "Value" "L"
+		(property "Value" "47uH"
 			(at 127 92.71 90)
 			(effects
@@
 			)
 		)
-		(property "Value" "R_Potentiometer"
+		(property "Value" "10kR"
 			(at 152.4 116.332 90)
 			(effects
@@
 			)
 		)
-		(property "Value" "R"
+		(property "Value" "330R"
 			(at 147.32 121.9199 0)
 			(effects
@@
 			)
 		)
-		(property "Value" "C"
+		(property "Value" "0.1uF"
 			(at 163.83 121.9199 0)
 			(effects
@@
 			)
 		)
-		(property "Value" "C"
+		(property "Value" "220uF"
 			(at 102.87 115.5699 0)
 			(effects

Commit message: added text
Other:
- note added: "Input"
- note added: "Output"
Changed lines of the file:
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@@
 	(generator_version "9.0")
 	(paper "A4")
+	(text "Output\n"
+		(exclude_from_sim no)
+		(at 218.948 111.252 0)
+		(effects
+			(font
+				(size 1.27 1.27)
+			)
+		)
+	)
+	(text "Input\n"
+		(exclude_from_sim no)
+		(at 72.898 173.228 0)
+		(effects
+			(font
+				(size 1.27 1.27)
+			)
+		)
+	)
 	(junction
 		(at 170.18 95.25)
