File: RouterSupplySwitcherSource/RouterSupplySwitcherSource.kicad_pcb (KiCad board)
At the start: 2 copper layers, 66 x 38 mm, 15 parts, among them J1 Barrel_Jack_Switch, J2 Barrel_Jack_Switch, J3 USB_A, P1 USB_C_Plug

Commit message: added values
Parts:
- C1: value C -> 220uF
- C2, C3: value C -> 0.1uF
- C4: value C -> 100uF
- D3: value D_Schottky_Dual_CommonAnode_AKK_Split -> SS34
- L1: value L -> 47uH
- R1: value R -> 330R
- RV1: value R_Potentiometer -> 10kR
Changed lines of the file:
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@@
 			)
 		)
-		(property "Value" "C"
+		(property "Value" "220uF"
 			(at 1 3.25 90)
 			(layer "F.Fab")
@@
 			)
 		)
-		(property "Value" "C"
+		(property "Value" "100uF"
 			(at 1 3.25 90)
 			(layer "F.Fab")
@@
 			)
 		)
-		(property "Value" "D_Schottky_Dual_CommonAnode_AKK_Split"
+		(property "Value" "SS34"
 			(at 6.557 5.111 90)
 			(layer "F.Fab")
@@
 			)
 		)
-		(property "Value" "L"
+		(property "Value" "47uH"
 			(at 0 6.35 0)
 			(layer "F.Fab")
@@
 			)
 		)
-		(property "Value" "R_Potentiometer"
+		(property "Value" "10kR"
 			(at -2.54 3.59 90)
 			(layer "F.Fab")
@@
 			)
 		)
-		(property "Value" "C"
+		(property "Value" "0.1uF"
 			(at 0 2.3 0)
 			(layer "F.Fab")
@@
 			)
 		)
-		(property "Value" "C"
+		(property "Value" "0.1uF"
 			(at 0 2.3 90)
 			(layer "F.Fab")
@@
 			)
 		)
-		(property "Value" "R"
+		(property "Value" "330R"
 			(at 5.08 2.37 0)
 			(layer "F.Fab")
